File: eagle/line_follower.brd (EAGLE design)
At the start: 100 x 80 mm, 41 parts, among them IC1 A4950, IC2 A4950, IC5 NCV4274CDT50RKG, J1 XT60PW-M, J2 2.54MM_HEADER_3X1, M1 N20-ENC2, M2 N20-ENC2, Q1 ALS-PT19-315C/L177/TR8, Q2 ALS-PT19-315C/L177/TR8, Q3 ALS-PT19-315C/L177/TR8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

Commit message: Another quarter-afternoon of layout
Parts:
- moved J2 38.6 mm to (12.7, 39.4), turned to 270 degrees
- moved J1 5.24 mm to (39.4, 66.0)
- moved R3 5.24 mm to (30.5, 20.3)
- moved R4 5.24 mm to (30.5, 25.4)
- moved R5 5.24 mm to (30.5, 30.5)
- moved R6 5.24 mm to (30.5, 35.6)
- moved R7 5.24 mm to (30.5, 40.6)
- moved C11 5.24 mm to (33.0, 43.2)
- moved C7 5.24 mm to (33.0, 22.9)
- moved C8 5.24 mm to (33.0, 27.9)
- moved C10 5.24 mm to (33.0, 38.1)
- moved C9 5.24 mm to (33.0, 33.0)
- moved C2 4.07 mm to (68.6, 10.8), flipped to the top, turned to 270 degrees
- moved X2 3.59 mm to (25.4, 66.0), turned to 0 degrees
- moved C4 3.59 mm to (68.6, 67.9), flipped to the top, turned to 270 degrees
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Connections:
- net ENCODER1A: now also X1.18; no longer X1.17
- net ENCODER1B: now also X1.17; no longer X1.18
Routing:
- net GND: track 154.0 -> 282.6 mm, vias 27 -> 86
- net ENCODER1A: track 20.8 -> 65.0 mm, vias 0 -> 1
- net ENCODER1B: track 23.9 -> 65.0 mm, vias 0 -> 1
- net GND1: track 17.8 -> 0.00 mm, vias 15 -> 0
- net VBAT: track 104.4 -> 114.2 mm, vias 4 -> 5
- net GND2: track 7.62 -> 0.00 mm, vias 5 -> 0
- net GND3: track 7.62 -> 0.00 mm, vias 5 -> 0
- net MOTOR1A: track 41.5 -> 46.7 mm, vias 0 -> 1
- net GND8: track 5.08 -> 0.00 mm, vias 11 -> 0
- net GND4: track 5.08 -> 0.00 mm, vias 3 -> 0
- net GND10: track 5.08 -> 0.00 mm, vias 3 -> 0
- net GND6: track 5.08 -> 0.00 mm, vias 3 -> 0
- net N$3: track 21.2 -> 24.3 mm
- net GND5: track 2.54 -> 0.00 mm, vias 11 -> 0
- net GND9: track 2.54 -> 0.00 mm, vias 1 -> 0
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
Commit message: Everything is connected on the board, but more work remains
Parts:
- moved LED1 67.9 mm to (12.7, 73.3), turned to 0 degrees
- moved LED6 67.9 mm to (12.7, 5.41), turned to 0 degrees
- moved J2 51.3 mm to (50.8, 5.08), turned to 0 degrees
- moved LED2 41.6 mm to (8.01, 60.1), turned to 0 degrees
- moved LED5 41.6 mm to (8.01, 18.6)
- moved R2 37.0 mm to (40.6, 66.0), turned to 180 degrees
- moved R1 33.2 mm to (45.7, 66.0), turned to 180 degrees
- moved C11 20.3 mm to (33.0, 22.9), flipped to the bottom, turned to 0 degrees
- moved C7 20.3 mm to (33.0, 43.2), flipped to the bottom, turned to 0 degrees
- moved R3 20.3 mm to (30.5, 40.6), flipped to the bottom, turned to 0 degrees
- moved R7 20.3 mm to (30.5, 20.3), flipped to the bottom, turned to 0 degrees
- moved LED3 14.0 mm to (5.63, 46.4)
- moved LED4 14.0 mm to (5.63, 32.4), turned to 0 degrees
- moved R4 10.2 mm to (30.5, 35.6), flipped to the bottom, turned to 0 degrees
- moved R6 10.2 mm to (30.5, 25.4), flipped to the bottom, turned to 0 degrees
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Connections:
- net +3V3: no longer IC1.4, IC2.4
- net +5V: now also IC1.4, IC2.4
- net LINE_LED0: now also LED1.A, LED2.C, LED5.A, LED6.C, X1.23; no longer LED1.C, LED2.A, LED5.C, LED6.A, X1.25
- net LINE_LED1: now also LED3.A, LED4.C, LED5.C, LED6.A; no longer LED1.A, LED2.C, LED3.C, LED4.A
- net LINE_LED2: now also LED1.C, LED2.A, LED3.C, LED4.A, X1.25; no longer LED3.A, LED4.C, LED5.A, LED6.C, X1.23
- net LINE_SENSOR0: now also X1.19; no longer X1.22
- net LINE_SENSOR1: now also X1.5; no longer X1.26
- net LINE_SENSOR3: now also X1.26; no longer X1.5
- net LINE_SENSOR4: now also X1.22; no longer X1.19
Routing:
- net +5V: track 3.62 -> 192.7 mm, vias 0 -> 5
- net GND: track 282.6 -> 406.0 mm, vias 86 -> 90
- net LINE_LED2: track 0.00 -> 84.7 mm, vias 0 -> 3
- net LINE_LED0: track 0.00 -> 82.2 mm, vias 0 -> 3
- net +3V3: track 105.5 -> 180.5 mm, vias 0 -> 1
- net LINE_LED1: track 0.00 -> 70.4 mm, vias 0 -> 3
- net LINE_SENSOR1: track 0.00 -> 67.4 mm, vias 0 -> 4
- net RANGE: track 0.00 -> 57.8 mm, vias 0 -> 1
- net BAT_SENSE: track 0.00 -> 55.6 mm, vias 0 -> 1
- net LINE_SENSOR4: track 0.00 -> 50.5 mm, vias 0 -> 2
- net LINE_SENSOR0: track 0.00 -> 47.6 mm, vias 0 -> 2
- net MOTOR0A: track 0.00 -> 47.6 mm
- net MOTOR0B: track 0.00 -> 47.0 mm
- net SDA: track 0.00 -> 42.7 mm, vias 0 -> 2
- net SCL: track 0.00 -> 39.9 mm, vias 0 -> 2
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Other:
- board text added: "2S-4S LiPo"
- board text removed: "3S LiPo"

Commit message: Layout complete, now a day or two for it to sink in and find more errors.
Parts:
- C1, C3: value 100uF 25V -> 100nF; device rcl:UD-6,3X5,8_NICHICON -> rcl:C0805
- C10, C11: value 100n -> 100uF 25V; device rcl:C0805 -> rcl:UD-6,3X5,8_NICHICON
- C4, C5: value 100nF -> 100n
- C6: value 22uF -> 100n
- C9: value 100n -> 22uF
- moved IC1 58.4 mm to (64.8, 68.6)
- moved IC2 58.4 mm to (64.8, 10.2)
- moved C2 57.1 mm to (68.6, 67.9)
- moved C3 50.3 mm to (68.6, 10.8), flipped to the top, turned to 270 degrees
- moved C10 45.8 mm to (64.8, 61.0), turned to 180 degrees
- moved C4 39.3 mm to (38.1, 43.2), flipped to the bottom, turned to 0 degrees
- moved M1 35.6 mm to (78.7, 57.1)
- moved M2 35.6 mm to (78.7, 21.6)
- moved C11 32.2 mm to (64.8, 17.8), turned to 180 degrees
- moved C9 27.4 mm to (59.7, 39.4), turned to 270 degrees
- moved C5 26.7 mm to (38.1, 38.1), turned to 0 degrees
- moved C6 22.5 mm to (38.1, 33.0), turned to 0 degrees
- moved C1 21.6 mm to (64.8, 39.4), turned to 270 degrees
- moved C7 16.1 mm to (38.1, 27.9)
- moved C8 16.1 mm to (38.1, 22.9)
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Connections:
- removed net ENCODER0A: M1.P$3, X1.7
- removed net ENCODER0B: M1.P$4, X1.6
- removed net MOTOR0A: IC1.3, X1.27
- removed net MOTOR0B: IC1.2, X1.28
- new net ENCODER2A: M2.P$3, X1.7
- new net ENCODER2B: M2.P$4, X1.6
- new net MOTOR2A: IC2.3, X1.27
- new net MOTOR2B: IC2.2, X1.28
- net +5V: now also C9.1; no longer C6.1
- net ENCODER1A: now also M1.P$4; no longer M2.P$4
- net ENCODER1B: now also M1.P$3; no longer M2.P$3
- net GND: now also C1.2, C10.-, C11.-, C3.2, C4.1, C5.1, C6.1, C9.2; no longer C1.-, C10.1, C11.1, C3.-, C4.2, C5.2, C6.2, C9.1
- net LINE_LED0: now also LED1.C, LED2.A, LED3.C, LED4.A; no longer LED1.A, LED2.C, LED5.A, LED6.C
- net LINE_LED1: now also LED1.A, LED2.C, LED5.A, LED6.C; no longer LED3.A, LED4.C, LED5.C, LED6.A
- net LINE_LED2: now also LED3.A, LED4.C, LED5.C, LED6.A; no longer LED1.C, LED2.A, LED3.C, LED4.A
- net LINE_SENSOR0: now also C4.2; no longer C7.2
- net LINE_SENSOR1: now also C5.2; no longer C8.2
- net LINE_SENSOR2: now also C6.2; no longer C9.2
- net LINE_SENSOR3: now also C7.2; no longer C10.2
- net LINE_SENSOR4: now also C8.2; no longer C11.2
- net MOTOR1A: now also IC1.2; no longer IC2.2
- net MOTOR1B: now also IC1.3; no longer IC2.3
- net VBAT: now also C1.1, C10.+, C11.+, C3.1; no longer C1.+, C3.+, C4.1, C5.1
Routing:
- net MOTOR0A: track 47.6 -> 0.00 mm
- net MOTOR0B: track 47.0 -> 0.00 mm
- net MOTOR2A: track 0.00 -> 45.0 mm
- net MOTOR2B: track 0.00 -> 44.5 mm
- net ENCODER0B: track 36.4 -> 0.00 mm
- net ENCODER0A: track 36.4 -> 0.00 mm
- net ENCODER2A: track 0.00 -> 33.9 mm
- net ENCODER2B: track 0.00 -> 33.9 mm
- net LINE_LED1: track 70.4 -> 85.8 mm, vias 3 -> 7
- net LINE_LED2: track 84.7 -> 70.0 mm, vias 3 -> 2
- net N$2: track 25.2 -> 13.7 mm
- net N$1: track 13.7 -> 25.2 mm
- net N$4: track 24.3 -> 14.2 mm
- net N$3: track 14.2 -> 24.3 mm
- net LINE_LED0: track 82.2 -> 72.4 mm, vias 3 -> 2
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- added copper zone on layer 1, net GND
- added copper zone on layer 16, net GND
