File: eagle/line_follower.sch (EAGLE design)
At the start: 39 parts, among them IC1 A4950, IC2 A4950, IC5 NCV4274CDT50RKG, J1 XT60PW-M, J2 2.54MM_HEADER_3X1, M1 N20-ENC2, M2 N20-ENC2, Q1 ALS-PT19-315C/L177/TR8, Q2 ALS-PT19-315C/L177/TR8, Q3 ALS-PT19-315C/L177/TR8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

Commit message: Layout complete, now a day or two for it to sink in and find more errors.
Parts:
- C1, C3: value 100uF 25V -> 100nF; device rcl:CPOL-EUUD-6,3X8,8 -> rcl:C-EUC0805
- C10, C11: value 100n -> 100uF 25V; device rcl:C-EUC0805 -> rcl:CPOL-EUUD-6,3X8,8
- C4, C5: value 100nF -> 100n
- C6: value 22uF -> 100n
- C9: value 100n -> 22uF
Connections:
- removed net ENCODER0A: M1.A, X1.IO17
- removed net ENCODER0B: M1.B, X1.IO16
- removed net MOTOR0A: IC1.IN1, X1.IO12
- removed net MOTOR0B: IC1.IN2, X1.IO13
- new net ENCODER2A: M2.A, X1.IO17
- new net ENCODER2B: M2.B, X1.IO16
- new net MOTOR2A: IC2.IN1, X1.IO12
- new net MOTOR2B: IC2.IN2, X1.IO13
- net +5V: now also C9.1; no longer C6.1
- net ENCODER1A: now also M1.B; no longer M2.B
- net ENCODER1B: now also M1.A; no longer M2.A
- net GND: now also C1.2, C10.-, C11.-, C3.2, C4.1, C5.1, C6.1, C9.2; no longer C1.-, C10.1, C11.1, C3.-, C4.2, C5.2, C6.2, C9.1
- net LINE_LED0: now also LED1.C, LED2.A, LED3.C, LED4.A; no longer LED1.A, LED2.C, LED5.A, LED6.C
- net LINE_LED1: now also LED1.A, LED2.C, LED5.A, LED6.C; no longer LED3.A, LED4.C, LED5.C, LED6.A
- net LINE_LED2: now also LED3.A, LED4.C, LED5.C, LED6.A; no longer LED1.C, LED2.A, LED3.C, LED4.A
- net LINE_SENSOR0: now also C4.2; no longer C7.2
- net LINE_SENSOR1: now also C5.2; no longer C8.2
- net LINE_SENSOR2: now also C6.2; no longer C9.2
- net LINE_SENSOR3: now also C7.2; no longer C10.2
- net LINE_SENSOR4: now also C8.2; no longer C11.2
- net MOTOR1A: now also IC1.IN2; no longer IC2.IN2
- net MOTOR1B: now also IC1.IN1; no longer IC2.IN1
- net VBAT: now also C1.1, C10.+, C11.+, C3.1; no longer C1.+, C3.+, C4.1, C5.1
Other:
- moved on the sheet: C2, C4, C5, C6, C7, C8, C9, IC1, IC2, LED1, LED2, LED3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
