File: kicad/line_follower.kicad_pcb (KiCad board)
At the start: 2 copper layers, 80 x 100 mm, 48 parts, among them J1 XT30PW-M, M1 MOTOR_ENC, M2 MOTOR_ENC, Q1 ALS-PT19-315C_L177_TR8, Q2 ALS-PT19-315C_L177_TR8, Q3 ALS-PT19-315C_L177_TR8, Q4 ALS-PT19-315C_L177_TR8, Q5 ALS-PT19-315C_L177_TR8, SW1 SW_Push, U1 A4950E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

Commit message: board: Manually fixed the outline to make step exporter happy
Other:
- outline, holes or cut-outs redrawn
Changed lines of the file:
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@@
   (general
     (thickness 1.6)
-    (drawings 59)
+    (drawings 64)
     (tracks 500)
     (zones 0)
@@
   (module cube-library:XT30PW-M (layer F.Cu)
     (at -31.75 45.72 180)
-    (fp_text reference J1 (at 0 -1.905 90) (layer F.SilkS)
+    (fp_text reference J1 (at -6.985 1.905 90) (layer F.SilkS)
       (effects (font (size 1 1) (thickness 0.15)))
     )
@@
     )
   )
+  (gr_line (start 38.854688 22.847512) (end 38.857868 22.845556) (layer Edge.Cuts) (width 0.001))
+  (gr_line (start 33.78982 81.254218) (end 33.846153 81.230769) (layer Edge.Cuts) (width 0.001))
+  (gr_line (start -39.999999 24.654889) (end -39.999999 24.655694) (layer Edge.Cuts) (width 0.001))
+  (gr_line (start -35 16.749999) (end -35 16.752716) (layer Edge.Cuts) (width 0.001))
+  (gr_line (start 38.85692 22.84476) (end 38.85692 22.84222) (layer F.Paste) (width 0.15))
   (gr_arc (start 30 6.999999) (end 30 11.999999) (angle -90) (layer F.SilkS) (width 0.2))
   (gr_line (start 35 6.999999) (end 35 -7) (layer F.SilkS) (width 0.2))
@@
     (effects (font (size 1.5 1.2) (thickness 0.25)) (justify left))
   )
-  (gr_line (start 39.999999 72) (end 39.999999 24.655694) (layer Edge.Cuts) (width 0.2))
-  (gr_arc (start -30 -7) (end -30 -12) (angle -90) (layer Edge.Cuts) (width 0.2))
-  (gr_line (start 30 -12) (end -30 -12) (layer Edge.Cuts) (width 0.2))
-  (gr_arc (start 30 -7) (end 35 -7) (angle -90) (layer Edge.Cuts) (width 0.2))
-  (gr_line (start 35 -7) (end 35 16.749999) (layer Edge.Cuts) (width 0.2))
-  (gr_arc (start 41.75 16.749999) (end 35 16.749999) (angle -64.62306647) (layer Edge.Cuts) (width 0.2))
-  (gr_arc (start 37.999999 24.655694) (end 39.999999 24.655694) (angle -64.62306647) (layer Edge.Cuts) (width 0.2))
-  (gr_arc (start 29.999999 72) (end 33.846153 81.230769) (angle -67.38013505) (layer Edge.Cuts) (width 0.2))
-  (gr_arc (start 0 0) (end -33.846153 81.230769) (angle -45.2397299) (layer Edge.Cuts) (width 0.2))
-  (gr_arc (start -29.999999 72) (end -39.999999 72) (angle -67.38013505) (layer Edge.Cuts) (width 0.2))
-  (gr_line (start -39.999999 72) (end -39.999999 24.655694) (layer Edge.Cuts) (width 0.2))
-  (gr_arc (start -37.999999 24.655694) (end -38.857142 22.848678) (angle -64.62306647) (layer Edge.Cuts) (width 0.2))
-  (gr_arc (start -41.75 16.749999) (end -38.857142 22.848678) (angle -64.62306647) (layer Edge.Cuts) (width 0.2))
-  (gr_line (start -35 -7) (end -35 16.749999) (layer Edge.Cuts) (width 0.2))
+  (gr_line (start 39.999998 71.996533) (end 39.999998 24.652227) (layer Edge.Cuts) (width 0.001))
+  (gr_arc (start -30 -7) (end -30 -12) (angle -90) (layer Edge.Cuts) (width 0.001))
+  (gr_line (start 30 -12) (end -30 -12) (layer Edge.Cuts) (width 0.001))
+  (gr_arc (start 30 -7) (end 35 -7) (angle -90) (layer Edge.Cuts) (width 0.001))
+  (gr_line (start 35 -7) (end 35 16.749999) (layer Edge.Cuts) (width 0.001))
+  (gr_arc (start 41.75 16.749999) (end 35 16.749999) (angle -64.6) (layer Edge.Cuts) (width 0.001))
+  (gr_arc (start 37.999998 24.652227) (end 39.999998 24.652227) (angle -64.6) (layer Edge.Cuts) (width 0.001))
+  (gr_arc (start 29.999999 72) (end 33.846153 81.230769) (angle -67.4) (layer Edge.Cuts) (width 0.001))
+  (gr_arc (start 0 0) (end -33.842952 81.232102) (angle -45.1977429) (layer Edge.Cuts) (width 0.001))
+  (gr_arc (start -29.999999 72) (end -39.999999 72) (angle -67.4) (layer Edge.Cuts) (width 0.001))
+  (gr_line (start -39.999999 72) (end -39.999999 24.655694) (layer Edge.Cuts) (width 0.001))
+  (gr_arc (start -37.999999 24.655694) (end -38.857142 22.848678) (angle -64.6) (layer Edge.Cuts) (width 0.001))
+  (gr_arc (start -41.75 16.749999) (end -38.857142 22.848678) (angle -64.6) (layer Edge.Cuts) (width 0.001))
+  (gr_line (start -35 -7) (end -35 16.749999) (layer Edge.Cuts) (width 0.001))
   (via (at -2.54 76.835) (size 1) (drill 0.5) (layers F.Cu B.Cu) (net 1))
   (via (at -11.43 76.2) (size 1) (drill 0.5) (layers F.Cu B.Cu) (net 1))
